File: Hardware/Qwiic GPS-RTK2 - ublox ZED-F9P.brd (EAGLE design)
At the start: 43.2 x 43.2 mm, 143 parts, among them J1 Radio, J2 Qwiic Right Angle, J3 PTH, J4 Qwiic Right Angle, U2 3.3V, U3 ZED-F9P

Commit message: Update caps to X7R. Change bead on RF input.
Parts:
- removed FRAME1: FRAME-LETTER, SparkFun-Aesthetics:CREATIVE_COMMONS
- added FRAME2: FRAME-LEDGER, SparkFun-Aesthetics:CREATIVE_COMMONS
- C1: device SparkFun-Capacitors:0603 -> SparkFun-Capacitors:0402
- FB1: value 120_OHM -> 120NH; device SparkFun-Coils:0402 -> SparkFun-Coils:0402_MURATA
- R14: value 10 -> 33
Connections:
- net ANT_VCC: now also FB1.P2; no longer FB1.2
- net GPS_ANT1: now also FB1.P1; no longer FB1.1
